File: BaterijaLodlaukums.sch (KiCad schematic (older format))
At the start: 2 parts

Commit message: BaterijaLodlaukums update to test GitHub Repo
Parts:
- added B3: BAT-BLH-001, Battery_Holder:BAT-BHL-001, symbol BaterijaLodlaukums-rescue:Battery_Holder_SMD1-Battery_Holder
- added B4: PC-027, Battery_Holder:PC-027, symbol BaterijaLodlaukums-rescue:Battery_Holder_SMD1-Battery_Holder
- added B5: CR2032, Battery_Holder:CR2025, symbol BaterijaLodlaukums-rescue:Battery_Holder_SMD1-Battery_Holder
- B1, B2: symbol Battery_Holder:Battery_Holder_SMD1 -> BaterijaLodlaukums-rescue:Battery_Holder_SMD1-Battery_Holder
Changed lines of the file:
@@
 $EndDescr
 $Comp
-L Battery_Holder:Battery_Holder_SMD1 B1
+L BaterijaLodlaukums-rescue:Battery_Holder_SMD1-Battery_Holder B1
 U 1 1 5E83747B
 P 5380 3900
@@
 $EndComp
 $Comp
-L Battery_Holder:Battery_Holder_SMD1 B2
+L BaterijaLodlaukums-rescue:Battery_Holder_SMD1-Battery_Holder B2
 U 1 1 5E837C48
 P 5390 3350
@@
 	1    0    0    -1
 $EndComp
+$Comp
+L BaterijaLodlaukums-rescue:Battery_Holder_SMD1-Battery_Holder B3
+U 1 1 5EA04182
+P 5400 2650
+F 0 "B3" H 5531 2946 50  0000 L CNN
+F 1 "BAT-BLH-001" H 5531 2855 50  0000 L CNN
+F 2 "Battery_Holder:BAT-BHL-001" H 5400 2650 50  0001 C CNN
+F 3 "http://cdn.sparkfun.com/datasheets/Prototyping/BAT-BLH-001.jpg" H 5400 2650 50  0001 C CNN
+	1    5400 2650
+	1    0    0    -1
+$EndComp
+$Comp
+L BaterijaLodlaukums-rescue:Battery_Holder_SMD1-Battery_Holder B4
+U 1 1 5EA042EF
+P 6650 2600
+F 0 "B4" H 6781 2896 50  0000 L CNN
+F 1 "PC-027" H 6781 2805 50  0000 L CNN
+F 2 "Battery_Holder:PC-027" H 6650 2600 50  0001 C CNN
+F 3 "https://www.lelong.com.my/cr2025-cr2032-battery-holder-2pcs-pkt-pc-027-yongmf83-187209081-2020-12-Sale-P.htm" H 6650 2600 50  0001 C CNN
+	1    6650 2600
+	1    0    0    -1
+$EndComp
+$Comp
+L BaterijaLodlaukums-rescue:Battery_Holder_SMD1-Battery_Holder B5
+U 1 1 5EA0577F
+P 6700 3250
+F 0 "B5" H 6831 3546 50  0000 L CNN
+F 1 "CR2032" H 6831 3455 50  0000 L CNN
+F 2 "Battery_Holder:CR2025" H 6700 3250 50  0001 C CNN
+F 3 "https://www.dx.com/p/jtron-bs-5-cr2032-cr2025-battery-holder-3v-motherboard-battery-holder-black-10-pcs-2036609.html#.XqBUdc1RVhE" H 6700 3250 50  0001 C CNN
+	1    6700 3250
+	1    0    0    -1
+$EndComp
